Commit message: Controlador y celda_pick_and_place
Cambiado controlador para que se cargue con la configuración en config y reescrito celda_pick_and_place.py

File: celda_descripcion/urdf/robot_celda_macro.xacro (robot description, xacro)
@@ -2,5 +2,4 @@
 <robot xmlns:xacro="http://ros.org/wiki/xacro">
   <xacro:include filename="$(find ur_description)/urdf/ur_macro.xacro"/>
-  <xacro:include filename="$(find onrobot_description)/urdf/onrobot_macro.xacro"/>
   <xacro:macro name="robot_celda" params="
     parent
@@ -82,5 +81,5 @@
     <!-- Efector final simulado en tool0 -->
     <!-- Ajustar más el cilindro para colisiones -->
-    <xacro:property name="gripper_len" value="0.21"/>
+    <!-- <xacro:property name="gripper_len" value="0.21"/>
     <link name="gripper">
       <visual>
@@ -110,5 +109,5 @@
       <child link="gripper_tip"/>
       <origin xyz="0 0 0.21" rpy="0 0 0"/>
-    </joint>
+    </joint> -->
     <!-- <link name="cable">
       <collision>
