Commit message: Cambiado wrist_3_joint a revolute {-pi, pi} para path tolerance violation y modificado posición parada_brida ya que estaba mal puesto anteriormente

File: celda_descripcion/urdf/robot_celda.urdf.xacro (robot description, xacro)
@@ -3,8 +3,8 @@
   <xacro:include filename="$(find celda_descripcion)/urdf/robot_celda_macro.xacro"/>
   <xacro:arg name="ur_type" default="ur3e"/>
-  <xacro:arg name="joint_limits_parameters_file" default="$(find ur_description)/config/$(arg ur_type)/joint_limits.yaml"/>
-  <xacro:arg name="kinematics_parameters_file" default="$(find ur_description)/config/$(arg ur_type)/default_kinematics.yaml"/>
-  <xacro:arg name="physical_parameters_file" default="$(find ur_description)/config/$(arg ur_type)/physical_parameters.yaml"/>
-  <xacro:arg name="visual_parameters_file" default="$(find ur_description)/config/$(arg ur_type)/visual_parameters.yaml"/>
+  <xacro:arg name="joint_limits_parameters_file" default="$(find celda_control)/config/$(arg ur_type)/joint_limits.yaml"/>
+  <xacro:arg name="kinematics_parameters_file" default="$(find celda_control)/config/$(arg ur_type)/default_kinematics.yaml"/>
+  <xacro:arg name="physical_parameters_file" default="$(find celda_control)/config/$(arg ur_type)/physical_parameters.yaml"/>
+  <xacro:arg name="visual_parameters_file" default="$(find celda_control)/config/$(arg ur_type)/visual_parameters.yaml"/>
   <link name="world"/>
   <!--This will create the scene where the robot is located in-->

File: celda_descripcion/urdf/robot_celda_macro.xacro (robot description, xacro)
@@ -81,9 +81,10 @@
     <!-- Efector final simulado en tool0 -->
     <!-- Ajustar más el cilindro para colisiones -->
-    <!-- <xacro:property name="gripper_len" value="0.21"/>
+    <xacro:property name="gripper_len" value="0.21"/>
+    <xacro:property name="gripper_radius" value="0.035"/>
     <link name="gripper">
       <visual>
         <geometry>
-          <cylinder radius="0.035" length="${gripper_len}"/>
+          <cylinder radius="${gripper_radius}" length="${gripper_len}"/>
         </geometry>
         <origin xyz="0 0 ${gripper_len/2}" rpy="0 0 0"/>
@@ -95,5 +96,5 @@
         <origin xyz="0 0 ${gripper_len/2}" rpy="0 0 0"/>
         <geometry>
-          <cylinder radius="0.035" length="${gripper_len}"/>
+          <cylinder radius="${gripper_radius}" length="${gripper_len}"/>
         </geometry>
       </collision>
@@ -108,19 +109,19 @@
       <parent link="gripper"/>
       <child link="gripper_tip"/>
-      <origin xyz="0 0 0.21" rpy="0 0 0"/>
-    </joint> -->
-    <!-- <link name="cable">
+      <origin xyz="0 0 ${gripper_len}" rpy="0 0 0"/>
+    </joint>
+    <link name="parada_brida">
       <collision>
         <geometry>
-          <sphere radius="0.03"/>
+          <sphere radius="${0.03 + gripper_radius}"/>
         </geometry>
         <origin xyz="0 0 0" rpy="0 0 0"/>
       </collision>
     </link>
-    <joint name="cable_joint" type="fixed">
-      <parent link="ur3e_tool0"/>
-      <child link="cable"/>
-      <origin xyz="0 -0.035 0.01" rpy="0 0 0"/>
-    </joint> -->
+    <joint name="parada_brida_joint" type="fixed">
+      <parent link="ur3e_flange"/>
+      <child link="parada_brida"/>
+      <origin xyz="0 0 0" rpy="0 0 0"/>
+    </joint>
   <!-- <xacro:onrobot onrobot_type="rg2" prefix=""/>
   <joint name="onrobot_base_link_joint" type="fixed">
